File: kicad/proj.kicad_pcb (KiCad board)
At the start: 2 copper layers, 254 x 127 mm, 65 parts, among them J1 USB-C, J2 OLED, J3 USB-A, SW1 SW_DIP_x01, SW10 SW_DIP_x01, SW11 SW_DIP_x01, SW12 SW_DIP_x01, SW13 SW_DIP_x01, SW14 SW_DIP_x01, SW15 SW_DIP_x01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

Commit message: adapt for LCSC part numbers
Parts:
- R3, R4: value 27 -> 22
- R9: value 390k -> 330k
- U3: value W25Q128JVS -> W25Q16JVSNIQ
- Y1: value ABM8-272-T3 -> X322512MOB4SI

Commit message: replace USB-A with top mount part
Parts:
- J3: footprint proj:USB-A-SMD_8-5-CB1-9ZB -> proj:USB-A-SMD_USB-M-21
- moved U5 1.49 mm to (188.4, 42.2)
- moved J3 0.66 mm to (188.4, 34.9)
Connections:
- J3 pad 6: (no net) -> GND
- J3 pad 7: (no net) -> GND
- J3 pad 8: (no net) -> GND
Routing:
- net +5V: track 47.4 -> 49.2 mm
- net /USB_A_P: track 25.3 -> 24.0 mm
- net /USB_A_N: track 25.4 -> 24.1 mm
- net GND: track 77.6 -> 78.2 mm
- net Net-(J3-D+): track 2.33 -> 2.93 mm
Other:
- outline, holes or cut-outs redrawn

Commit message: add acrylic layouts
Parts:
- moved SW21 4.12 mm to (144.0, 37.3), turned to -90 degrees
- moved R9 2.74 mm to (241.7, 43.4)
- moved C19 2.74 mm to (250.7, 43.4)
- moved C20 2.74 mm to (248.5, 43.4)
- moved C21 2.74 mm to (249.5, 43.4)
- moved C22 2.74 mm to (240.1, 42.7)
- moved C23 2.74 mm to (238.0, 42.7)
- moved J2 2.74 mm to (245.0, 46.5)
- moved C18 2.74 mm to (251.8, 43.5)
- moved C10 1.80 mm to (166.6, 43.4)
- moved C6 1.80 mm to (156.1, 43.4)
- moved R12 1.80 mm to (154.4, 35.2)
- moved R2 1.80 mm to (152.4, 35.2)
- moved R6 1.80 mm to (155.6, 32.1)
- moved SW1 1.80 mm to (110.0, 47.6)
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Connections:
- J2 pad 18: /GPIO18 -> /GPIO19
- J2 pad 19: /GPIO19 -> /GPIO18
- J2 pad 20: /GPIO19 -> /GPIO18
- SW21 pad 1: GND -> Net-(R2-Pad1)
- SW21 pad 2: Net-(R2-Pad1) -> GND
Routing:
- net /GPIO18: track 84.5 -> 91.4 mm
- net /GPIO19: track 86.9 -> 91.8 mm
- net Net-(R2-Pad1): track 2.70 -> 6.82 mm
- net +3V3: track 137.5 -> 135.4 mm
- net /GPIO20: track 100.5 -> 101.5 mm
- net /GPIO21: track 81.7 -> 82.7 mm
